File: hardware/power-meter.kicad_pcb (KiCad board)
At the start: 4 copper layers, 45 x 30 mm, 30 parts, among them J1 USB_C_Receptacle_USB2.0_16P, J2 USB_C_Receptacle_USB2.0_16P, J3 OLED, J4 PROG, J5 IN+, J6 IN-, J7 OUT+, J8 OUT-, SW1 SW_Push, SW2 SW_Push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

Commit message: --
Routing:
- net GND: track 4.51 -> 9.95 mm, vias 18 -> 14
Changed lines of the file:
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@@
+	)
+	(segment
+		(start 149.685 73.2675)
+		(end 149.685 73.8075)
+		(width 0.5)
+		(layer "F.Cu")
+		(net 1)
 	)
 	(segment
@@
 	)
 	(segment
+		(start 149.685 66.8675)
+		(end 149.685 66.3275)
+		(width 0.5)
+		(layer "F.Cu")
+		(net 1)
+	)
+	(segment
+		(start 118.435 73.7825)
+		(end 117.855 74.3625)
+		(width 0.5)
+		(layer "F.Cu")
+		(net 1)
+	)
+	(segment
+		(start 149.685 73.8075)
+		(end 150.265 74.3875)
+		(width 0.5)
+		(layer "F.Cu")
+		(net 1)
+	)
+	(segment
+		(start 118.435 66.3025)
+		(end 117.855 65.7225)
+		(width 0.5)
+		(layer "F.Cu")
+		(net 1)
+	)
+	(segment
+		(start 118.435 66.8425)
+		(end 118.435 66.3025)
+		(width 0.5)
+		(layer "F.Cu")
+		(net 1)
+	)
+	(segment
 		(start 143.25 70.5675)
 		(end 143.26 70.5575)
@@
 	)
 	(segment
+		(start 149.685 66.3275)
+		(end 150.265 65.7475)
+		(width 0.5)
+		(layer "F.Cu")
+		(net 1)
+	)
+	(segment
 		(start 137.5 73.5575)
 		(end 137.53 73.5875)
@@
 	)
 	(segment
+		(start 118.435 73.2425)
+		(end 118.435 73.7825)
+		(width 0.5)
+		(layer "F.Cu")
+		(net 1)
+	)
+	(segment
 		(start 130.795 62.7325)
 		(end 132.255 62.7325)
@@
 	)
 	(via
-		(at 119.39 66.3975)
+		(at 127.16 70.1125)
 		(size 0.45)
 		(drill 0.3)
@@
 	)
 	(via
-		(at 127.16 70.1125)
+		(at 122.985 65.2125)
+		(size 0.45)
+		(drill 0.3)
+		(layers "F.Cu" "B.Cu")
+		(net 1)
+	)
+	(via
+		(at 146.155 76.2375)
+		(size 0.45)
+		(drill 0.3)
+		(layers "F.Cu" "B.Cu")
+		(net 1)
+	)
+	(via
+		(at 121.235 67.4875)
+		(size 0.45)
+		(drill 0.3)
+		(layers "F.Cu" "B.Cu")
+		(net 1)
+	)
+	(via
+		(at 139.85 65.8275)
 		(size 0.45)
 		(drill 0.3)
@@
 	)
 	(via
-		(at 122.985 65.2125)
-		(size 0.45)
-		(drill 0.3)
-		(layers "F.Cu" "B.Cu")
-		(net 1)
-	)
-	(via
-		(at 146.155 76.2375)
-		(size 0.45)
-		(drill 0.3)
-		(layers "F.Cu" "B.Cu")
-		(net 1)
-	)
-	(via
-		(at 121.235 67.4875)
-		(size 0.45)
-		(drill 0.3)
-		(layers "F.Cu" "B.Cu")
-		(net 1)
-	)
-	(via
-		(at 139.85 65.8275)
+		(at 143.25 70.5675)
 		(size 0.45)
 		(drill 0.3)
@@
 	)
 	(via
-		(at 143.25 70.5675)
+		(at 137.53 73.5875)
 		(size 0.45)
 		(drill 0.3)
@@
 	)
 	(via
-		(at 137.53 73.5875)
+		(at 128.22 70.8875)
 		(size 0.45)
 		(drill 0.3)
@@
 	)
 	(via
-		(at 128.22 70.8875)
+		(at 132.92 75.9575)
+		(size 0.45)
+		(drill 0.3)
+		(layers "F.Cu" "B.Cu")
+		(net 1)
+	)
+	(via
+		(at 134.5 73.513592)
 		(size 0.45)
 		(drill 0.3)
@@
 	)
 	(via
-		(at 148.65 66.8675)
-		(size 0.45)
-		(drill 0.3)
-		(layers "F.Cu" "B.Cu")
-		(free yes)
-		(net 1)
-	)
-	(via
-		(at 132.92 75.9575)
-		(size 0.45)
-		(drill 0.3)
-		(layers "F.Cu" "B.Cu")
-		(net 1)
-	)
-	(via
-		(at 134.5 73.513592)
-		(size 0.45)
-		(drill 0.3)
-		(layers "F.Cu" "B.Cu")
-		(free yes)
-		(net 1)
-	)
-	(via
 		(at 131.37 75.9575)
 		(size 0.45)
@@
 	)
 	(via
-		(at 119.79 73.4275)
-		(size 0.45)
-		(drill 0.3)
-		(layers "F.Cu" "B.Cu")
-		(free yes)
-		(net 1)
-	)
-	(via
 		(at 131.39 68.1675)
-		(size 0.45)
-		(drill 0.3)
-		(layers "F.Cu" "B.Cu")
-		(free yes)
-		(net 1)
-	)
-	(via
-		(at 148.65 73.2775)
 		(size 0.45)
 		(drill 0.3)
@@
 	)
 	(segment
+		(start 130.745 73.7825)
+		(end 131.37 74.4075)
+		(width 0.3)
+		(layer "F.Cu")
+		(net 15)
+	)
+	(segment
 		(start 138.4325 64.345)
 		(end 139.195 65.1075)
@@
 	)
 	(segment
-		(start 130.745 73.7825)
-		(end 131.37 74.4075)
+		(start 130.745 72.5825)
+		(end 130.745 73.7825)
 		(width 0.3)
 		(layer "F.Cu")
@@
 		(width 0.3)
 		(layer "F.Cu")
-		(net 15)
-	)
-	(segment
-		(start 130.745 72.5825)
-		(end 130.745 73.7825)
-		(width 0.3)
-		(layer "F.Cu")

Commit message: --
Routing:
- net Net-(J1-CC1): track 12.6 -> 13.9 mm
- net Net-(R7-Pad1): track 35.2 -> 36.0 mm
Changed lines of the file:
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@@
 			(outputformat 1)
 			(mirror no)
-			(drillshape 1)
+			(drillshape 0)
 			(scaleselection 1)
-			(outputdirectory "")
+			(outputdirectory "/Users/snakeye/Downloads/power-meter")
 		)
 	)
@@
 	)
 	(segment
-		(start 123.532947 68.854553)
-		(end 119.728734 68.854553)
+		(start 122.41 69.9775)
+		(end 120.851681 69.9775)
 		(width 0.2)
 		(layer "B.Cu")
@@
 	)
 	(segment
-		(start 128.005 64.3825)
-		(end 123.532947 68.854553)
+		(start 120.851681 69.9775)
+		(end 119.728734 68.854553)
 		(width 0.2)
 		(layer "B.Cu")
@@
 	(segment
 		(start 129.245 64.3825)
-		(end 128.005 64.3825)
+		(end 129.245 65.106814)
+		(width 0.2)
+		(layer "B.Cu")
+		(net 2)
+	)
+	(segment
+		(start 128.904314 65.4475)
+		(end 126.94 65.4475)
+		(width 0.2)
+		(layer "B.Cu")
+		(net 2)
+	)
+	(segment
+		(start 129.245 65.106814)
+		(end 128.904314 65.4475)
+		(width 0.2)
+		(layer "B.Cu")
+		(net 2)
+	)
+	(segment
+		(start 126.94 65.4475)
+		(end 122.41 69.9775)
 		(width 0.2)
 		(layer "B.Cu")
@@
 	)
 	(segment
-		(start 119.63 71.5375)
-		(end 121.912947 69.254553)
+		(start 129.07 65.8475)
+		(end 130.535 64.3825)
 		(width 0.2)
 		(layer "B.Cu")
@@
 	)
 	(segment
-		(start 128.045686 64.9075)
-		(end 130.27 64.9075)
+		(start 127.105686 65.8475)
+		(end 129.07 65.8475)
 		(width 0.2)
 		(layer "B.Cu")
@@
 	)
 	(segment
-		(start 123.698633 69.254553)
-		(end 128.045686 64.9075)
+		(start 130.535 64.3825)
+		(end 130.795 64.3825)
 		(width 0.2)
 		(layer "B.Cu")
@@
 	)
 	(segment
-		(start 121.912947 69.254553)
-		(end 123.698633 69.254553)
+		(start 119.63 71.5375)
+		(end 120.79 70.3775)
 		(width 0.2)
 		(layer "B.Cu")
@@
 	)
 	(segment
-		(start 130.27 64.9075)
-		(end 130.795 64.3825)
+		(start 120.79 70.3775)
+		(end 122.575686 70.3775)
+		(width 0.2)
+		(layer "B.Cu")
+		(net 7)
+	)
+	(segment
+		(start 122.575686 70.3775)
+		(end 127.105686 65.8475)
 		(width 0.2)
 		(layer "B.Cu")
@@
 	)
 	(segment
-		(start 146.585 73.515037)
-		(end 141.285 78.815037)
+		(start 146.585 70.600037)
+		(end 146.585 72.4625)
 		(width 0.2)
 		(layer "B.Cu")
@@
 	)
 	(segment
-		(start 146.585 69.7425)
-		(end 146.585 73.515037)
+		(start 141.285 77.7625)
+		(end 141.285 81.8375)
 		(width 0.2)
 		(layer "B.Cu")
@@
 	)
 	(segment
-		(start 141.285 78.815037)
-		(end 141.285 81.8375)
+		(start 144.935 70.2925)
+		(end 146.277463 70.2925)
+		(width 0.2)
+		(layer "B.Cu")
+		(net 39)
+	)
+	(segment
+		(start 146.277463 70.2925)
+		(end 146.585 70.600037)
+		(width 0.2)
+		(layer "B.Cu")
+		(net 39)
+	)
+	(segment
+		(start 146.585 72.4625)
+		(end 141.285 77.7625)
 		(width 0.2)
 		(layer "B.Cu")
@@
 	(segment
 		(start 140.98 64.1375)
-		(end 146.585 69.7425)
+		(end 140.98 66.3375)
+		(width 0.2)
+		(layer "B.Cu")
+		(net 39)
+	)
+	(segment
+		(start 140.98 66.3375)
+		(end 144.935 70.2925)
 		(width 0.2)
 		(layer "B.Cu")
@@
 	)
 	(segment
+		(start 142.535 71.5475)
+		(end 135.37 64.3825)
+		(width 0.2)
+		(layer "B.Cu")
+		(net 52)
+	)
+	(segment
 		(start 136.04 58.4615)
 		(end 135.231 57.6525)
@@
 	)
 	(segment
-		(start 142.695 71.7075)
-		(end 135.37 64.3825)
+		(start 146.04 71.7075)
+		(end 145.88 71.5475)
 		(width 0.2)
 		(layer "B.Cu")
@@
 	)
 	(segment
-		(start 136.04 63.7125)
-		(end 136.04 58.4615)
+		(start 145.88 71.5475)
+		(end 142.535 71.5475)
 		(width 0.2)
 		(layer "B.Cu")
@@
 	)
 	(segment
-		(start 146.04 71.7075)
-		(end 142.695 71.7075)
+		(start 136.04 63.7125)
+		(end 136.04 58.4615)
 		(width 0.2)
 		(layer "B.Cu")
@@
 	)
 	(segment
-		(start 136.415343 63.902843)
-		(end 136.44 63.878186)
+		(start 137.135 57.7825)
+		(end 137.135 57.6525)
 		(width 0.2)
 		(layer "B.Cu")
@@
 	)
 	(segment
-		(start 136.895 65.341814)
-		(end 136.895 64.3825)
+		(start 136.44 58.4775)
+		(end 137.135 57.7825)
 		(width 0.2)
 		(layer "B.Cu")
@@
 	)
 	(segment
-		(start 142.860686 71.3075)
-		(end 136.895 65.341814)
+		(start 136.44 63.878186)
+		(end 136.44 58.4775)
 		(width 0.2)
 		(layer "B.Cu")
@@
 	)
 	(segment
-		(start 146.06 70.8175)
-		(end 145.57 71.3075)
+		(start 136.895 64.3825)
+		(end 136.415343 63.902843)
 		(width 0.2)
 		(layer "B.Cu")
@@
 	)
 	(segment
-		(start 136.44 58.3475)
-		(end 137.135 57.6525)
+		(start 142.700686 71.1475)
+		(end 136.895 65.341814)
 		(width 0.2)
 		(layer "B.Cu")
@@
 	)
 	(segment
-		(start 136.895 64.3825)
-		(end 136.415343 63.902843)
+		(start 136.895 65.341814)
+		(end 136.895 64.3825)
 		(width 0.2)
 		(layer "B.Cu")
@@
 	)
 	(segment
-		(start 136.44 63.878186)
-		(end 136.44 58.3475)
+		(start 145.73 71.1475)
+		(end 142.700686 71.1475)
+		(width 0.2)
+		(layer "B.Cu")
+		(net 54)
+	)
+	(segment
+		(start 146.06 70.8175)
+		(end 145.73 71.1475)
 		(width 0.2)
 		(layer "B.Cu")
@@
 	)
 	(segment
-		(start 145.57 71.3075)
-		(end 142.860686 71.3075)
+		(start 136.415343 63.902843)
+		(end 136.44 63.878186)
 		(width 0.2)
 		(layer "B.Cu")

Commit message: OLED power fixed
Connections:
- J3 pad 1: +3.3V -> GND
- J3 pad 2: GND -> +3.3V
Changed lines of the file:
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@@
 			(drillshape 0)
 			(scaleselection 1)
-			(outputdirectory "/Users/snakeye/Downloads/power-meter")
+			(outputdirectory "/Users/snakeye/Downloads/power-meter-v1")
 		)
 	)
@@
 			(layers "*.Cu" "*.Mask")
 			(remove_unused_layers no)
-			(net 15 "+3.3V")
+			(net 1 "GND")
 			(pinfunction "Pin_1")
 			(pintype "passive")
@@
 			(layers "*.Cu" "*.Mask")
 			(remove_unused_layers no)
-			(net 1 "GND")
+			(net 15 "+3.3V")
 			(pinfunction "Pin_2")
 			(pintype "passive")

Commit message: --
Parts:
- moved C1 4.15 mm to (123.0, 72.0), turned to -90 degrees
Routing:
- net VBUS: track 34.6 -> 38.0 mm
- net /NRST: track 26.0 -> 24.6 mm
- net +5V: track 49.5 -> 48.8 mm
- net GND: vias 14 -> 18

Commit message: feat: v2
Consolidate all work related to hardware revision v2 and firmware migration for that revision.

Hardware scope:

- Redesign PCB/schematic from v1 to v2 with updated component and connectivity decisions.

- Add STM32G431 symbol/library assets used by the new design.

- Integrate board-level corrections performed after first v2 routing pass.

Firmware scope:

- Migrate firmware target to STM32G431 platform and board configuration.

- Update build configuration and platform definitions for the new MCU/board.

- Adapt application logic to v2 hardware behavior and interfaces.

- Refactor firmware from monolithic source into focused modules (adc/config/display/util).

- Apply stabilization fixes after modular split.

Why:

- Represent v2 as a coherent generation change (hardware redesign + firmware migration).

- Keep migration rationale and resulting architecture in one clear historical checkpoint.
Parts:
- removed J5: IN+, Connector_PinSocket_2.54mm:PinSocket_1x01_P2.54mm_Vertical
- removed J6: IN-, Connector_PinSocket_2.54mm:PinSocket_1x01_P2.54mm_Vertical
- removed J7: OUT+, Connector_PinSocket_2.54mm:PinSocket_1x01_P2.54mm_Vertical
- removed J8: OUT-, Connector_PinSocket_2.54mm:PinSocket_1x01_P2.54mm_Vertical
- added C10: 1uF, Capacitor_SMD:C_0603_1608Metric, F.Cu at (125.8, 66.9)
- added C11: 0.1uF, Capacitor_SMD:C_0603_1608Metric, F.Cu at (136.3, 61.4)
- added C12: 22uF, Capacitor_SMD:C_0603_1608Metric, F.Cu at (128.1, 69.2)
- added C13: 1uF, Capacitor_SMD:C_0603_1608Metric, F.Cu at (115.2, 57.1)
- added C14: 1uF, Capacitor_SMD:C_0603_1608Metric, F.Cu at (116.8, 57.1)
- added R10: 2, Resistor_SMD:R_0603_1608Metric, F.Cu at (125.0, 69.2)
- added R11: 2, Resistor_SMD:R_0603_1608Metric, F.Cu at (126.5, 69.2)
- added R8: 56k, Resistor_SMD:R_0603_1608Metric, F.Cu at (142.7, 76.7)
- added R9: 56k, Resistor_SMD:R_0603_1608Metric, F.Cu at (141.1, 76.7)
- added U5: REF5045AD, Package_SO:SOIC-8_3.9x4.9mm_P1.27mm, F.Cu at (116.0, 61.5)
- added U6: M24C02-FMN, Package_SO:SOIC-8_3.9x4.9mm_P1.27mm, F.Cu at (152.1, 61.4)
- U2: value STM32F103CBTx -> STM32G431C8Tx
- moved C8 24.2 mm to (125.8, 62.0)
- moved C4 16.8 mm to (142.5, 61.4), turned to 90 degrees
- moved C5 16.8 mm to (141.0, 61.4), turned to 90 degrees
- moved R6 14.3 mm to (139.6, 76.7), turned to -90 degrees
- moved C6 14.3 mm to (138.0, 76.7), turned to -90 degrees
- moved R7 14.0 mm to (134.9, 76.7)
- moved C7 13.2 mm to (136.5, 76.7), turned to -90 degrees
- moved C9 12.5 mm to (127.6, 77.3), turned to -90 degrees
- moved U1 8.89 mm to (124.3, 77.2)
- moved R1 7.77 mm to (121.5, 62.7)
- moved R2 7.77 mm to (123.1, 62.7)
- moved U3 7.59 mm to (125.8, 64.5)
- moved U4 6.01 mm to (130.1, 63.8)
- moved C3 5.74 mm to (129.6, 69.2)
- moved C1 5.52 mm to (121.3, 77.3)
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Connections:
- J2 pad A5: unconnected-(J2-CC1-PadA5) -> Net-(J2-CC1)
- J2 pad A6: /D+ -> unconnected-(J2-D+-PadA6)
- J2 pad A7: /D- -> unconnected-(J2-D--PadA7)
- J2 pad B5: unconnected-(J2-CC2-PadB5) -> Net-(J2-CC2)
- J2 pad B6: /D+ -> unconnected-(J2-D+-PadB6)
- J2 pad B7: /D- -> unconnected-(J2-D--PadB7)
- U2 pad 14: /CS -> unconnected-(U2-PA6-Pad14)
- U2 pad 15: /SCK -> unconnected-(U2-PA7-Pad15)
- U2 pad 16: /MISO -> unconnected-(U2-PB0-Pad16)
- U2 pad 17: /MOSI -> unconnected-(U2-PB1-Pad17)
- U2 pad 18: /DRDY -> unconnected-(U2-PB2-Pad18)
- U2 pad 19: /BUTTON1 -> GND
- U2 pad 20: /BUTTON2 -> +3.3V
- U2 pad 21: unconnected-(U2-PB10-Pad21) -> +3.3V
- U2 pad 29: unconnected-(U2-PA8-Pad29) -> /DRDY
- U2 pad 30: unconnected-(U2-PA9-Pad30) -> /SDA
- U2 pad 31: unconnected-(U2-PA10-Pad31) -> /SCL
- U2 pad 33: unconnected-(U2-PA12-Pad33) -> /D-
- U2 pad 34: /SWDIO -> /D+
- U2 pad 37: /SWCLK -> /SWDIO
- U2 pad 38: unconnected-(U2-PA15-Pad38) -> /SWCLK
- U2 pad 39: unconnected-(U2-PB3-Pad39) -> /CS
- U2 pad 40: unconnected-(U2-PB4-Pad40) -> /SCK
- U2 pad 41: unconnected-(U2-PB5-Pad41) -> /MISO
- U2 pad 42: /SCL -> /MOSI
- U2 pad 43: /SDA -> unconnected-(U2-PB6-Pad43)
- U2 pad 44: GND -> /BUTTON1
- U2 pad 45: unconnected-(U2-PB8-Pad45) -> GND
- U2 pad 46: unconnected-(U2-PB9-Pad46) -> /BUTTON2
- U2 pad 8: GND -> unconnected-(U2-PA0-Pad8)
- U2 pad 9: +3.3V -> unconnected-(U2-PA1-Pad9)
- U3 pad 4: VBUS -> Net-(U3-IN+)
- U3 pad 5: +5V -> Net-(U3-IN-)
- U4 pad 10: unconnected-(U4-AIN1-Pad10) -> /ADC_IN
- U4 pad 11: /ADC_IN -> /VREF
- U4 pad 6: unconnected-(U4-AIN3/REFN1-Pad6) -> GND
- U4 pad 8: unconnected-(U4-REFN0-Pad8) -> GND
- U4 pad 9: unconnected-(U4-REFP0-Pad9) -> /VREF
Routing:
- net /VREF: track 0.00 -> 22.4 mm, vias 0 -> 2
- net Net-(R7-Pad1): track 36.4 -> 17.4 mm
- net /NRST: track 24.6 -> 8.69 mm
- net Net-(J2-CC2): track 0.00 -> 14.3 mm, vias 0 -> 2
- net /D-: track 38.3 -> 24.7 mm
- net /D+: track 38.0 -> 26.1 mm
- net Net-(J2-CC1): track 0.00 -> 10.8 mm, vias 0 -> 2
- net GND: track 9.95 -> 0.00 mm, vias 18 -> 17
- net /DRDY: track 5.54 -> 12.4 mm
- net /SWCLK: track 14.1 -> 20.6 mm
- net Net-(J1-CC1): track 13.9 -> 7.77 mm
- net /CS: track 7.20 -> 11.4 mm
- net /SCK: track 5.08 -> 9.22 mm
- net Net-(J1-CC2): track 15.4 -> 12.0 mm
- net Net-(U3-IN+): track 0.00 -> 3.04 mm
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